Commit message: create bot_one shape

File: description/robot_core.xacro (robot description, xacro)
@@ -27,5 +27,5 @@
             <origin xyz="0.15 0 0.075"/>
             <geometry>
-                <box size="0.3 0.3 0.15"/>
+                <box size="0.5 0.3 0.15"/>
             </geometry>
             <material name="white"/>
@@ -41,12 +41,12 @@
         </xacro:inertial_box>
     </link>
-    <!-- LEFT WHEEL LINK -->
-    <joint name="left_wheel_joint" type="continuous">
+    <!-- LEFT WHEEL FRONT LINK -->
+    <joint name="left_wheel_joint_front" type="continuous">
         <parent link="base_link"/>
-        <child link="left_wheel"/>
-        <origin xyz="0 0.175 0" rpy="-${pi/2} 0 0"/>
+        <child link="left_wheel_front"/>
+        <origin xyz="0.2 0.175 0" rpy="-${pi/2} 0 0"/>
         <axis xyz="0 0 1"/>
     </joint>
-    <link name="left_wheel">
+    <link name="left_wheel_front">
         <visual>
             <geometry>
@@ -64,12 +64,12 @@
         </xacro:inertial_cylinder>
     </link>
-    <!-- RIGHT WHEEL LINK -->
-    <joint name="right_wheel_joint" type="continuous">
+    <!-- LEFT WHEEL BACK LINK -->
+    <joint name="left_wheel_joint_back" type="continuous">
         <parent link="base_link"/>
-        <child link="right_wheel"/>
-        <origin xyz="0 -0.175 0" rpy="${pi/2} 0 0"/>
-        <axis xyz="0 0 -1"/>
+        <child link="left_wheel_back"/>
+        <origin xyz="-0.1 0.175 0" rpy="-${pi/2} 0 0"/>
+        <axis xyz="0 0 1"/>
     </joint>
-    <link name="right_wheel">
+    <link name="left_wheel_back">
         <visual>
             <geometry>
@@ -87,25 +87,49 @@
         </xacro:inertial_cylinder>
     </link>
-    <!-- CASTER WHEEL LINK -->
-    <joint name="caster_wheel_joint" type="fixed">
-        <parent link="chassis"/>
-        <child link="caster_wheel"/>
-        <origin xyz="0.24 0 0"/>
+    <!-- RIGHT WHEEL FRONT LINK -->
+    <joint name="right_wheel_joint_front" type="continuous">
+        <parent link="base_link"/>
+        <child link="right_wheel_front"/>
+        <origin xyz="0.2 -0.175 0" rpy="${pi/2} 0 0"/>
+        <axis xyz="0 0 -1"/>
     </joint>
-    <link name="caster_wheel">
+    <link name="right_wheel_front">
         <visual>
             <geometry>
-                <sphere radius="0.05"/>
+                <cylinder radius="0.05" length="0.04"/>
             </geometry>
-            <material name="black"/>
+            <material name="blue"/>
         </visual>
         <collision>
             <geometry>
-                <sphere radius="0.05"/>
+                <cylinder radius="0.05" length="0.04"/>
             </geometry>
         </collision>
-        <xacro:inertial_sphere mass='0.1' radius="0.05">
+        <xacro:inertial_cylinder mass="0.1" length="0.04" radius="0.05">
             <origin xyz="0 0 0" rpy="0 0 0"/>
-        </xacro:inertial_sphere>
+        </xacro:inertial_cylinder>
+    </link>
+    <!-- RIGHT WHEEL BACK LINK -->
+    <joint name="right_wheel_joint_back" type="continuous">
+        <parent link="base_link"/>
+        <child link="right_wheel_back"/>
+        <origin xyz="-0.1 -0.175 0" rpy="${pi/2} 0 0"/>
+        <axis xyz="0 0 -1"/>
+    </joint>
+    <link name="right_wheel_back">
+        <visual>
+            <geometry>
+                <cylinder radius="0.05" length="0.04"/>
+            </geometry>
+            <material name="blue"/>
+        </visual>
+        <collision>
+            <geometry>
+                <cylinder radius="0.05" length="0.04"/>
+            </geometry>
+        </collision>
+        <xacro:inertial_cylinder mass="0.1" length="0.04" radius="0.05">
+            <origin xyz="0 0 0" rpy="0 0 0"/>
+        </xacro:inertial_cylinder>
     </link>
 </robot>
