Commit message: driver control

File: description/robot.urdf.xacro (robot description, xacro)
@@ -2,3 +2,4 @@
 <robot xmlns:xacro="http://www.ros.org/wiki/xacro"  name="robot">
     <xacro:include filename="robot_core.xacro" />
+    <xacro:include filename="gazebo_control.xacro" />
 </robot>

File: description/robot_core.xacro (robot description, xacro)
@@ -41,4 +41,7 @@
         </xacro:inertial_box>
     </link>
+    <gazebo reference="chassis">
+        <material>Gazebo/White</material>
+    </gazebo>
     <!-- LEFT WHEEL FRONT LINK -->
     <joint name="left_wheel_joint_front" type="continuous">
@@ -64,12 +67,15 @@
         </xacro:inertial_cylinder>
     </link>
-    <!-- LEFT WHEEL BACK LINK -->
-    <joint name="left_wheel_joint_back" type="continuous">
-        <parent link="base_link"/>
-        <child link="left_wheel_back"/>
+    <gazebo reference="left_wheel_front">
+        <material>Gazebo/Blue</material>
+    </gazebo>
+    <!-- LEFT WHEEL REAR LINK -->
+    <joint name="left_wheel_joint_rear" type="fixed">
+        <parent link="chassis"/>
+        <child link="left_wheel_rear"/>
         <origin xyz="-0.1 0.175 0" rpy="-${pi/2} 0 0"/>
         <axis xyz="0 0 1"/>
     </joint>
-    <link name="left_wheel_back">
+    <link name="left_wheel_rear">
         <visual>
             <geometry>
@@ -87,4 +93,9 @@
         </xacro:inertial_cylinder>
     </link>
+    <gazebo reference="left_wheel_rear">
+        <material>Gazebo/Blue</material>
+        <mu1 value="0.001"/>
+        <mu2 value="0.001"/>
+    </gazebo>
     <!-- RIGHT WHEEL FRONT LINK -->
     <joint name="right_wheel_joint_front" type="continuous">
@@ -110,12 +121,15 @@
         </xacro:inertial_cylinder>
     </link>
-    <!-- RIGHT WHEEL BACK LINK -->
-    <joint name="right_wheel_joint_back" type="continuous">
-        <parent link="base_link"/>
-        <child link="right_wheel_back"/>
+    <gazebo reference="right_wheel_front">
+        <material>Gazebo/Blue</material>
+    </gazebo>
+    <!-- RIGHT WHEEL REAR LINK -->
+    <joint name="right_wheel_joint_rear" type="fixed">
+        <parent link="chassis"/>
+        <child link="right_wheel_rear"/>
         <origin xyz="-0.1 -0.175 0" rpy="${pi/2} 0 0"/>
         <axis xyz="0 0 -1"/>
     </joint>
-    <link name="right_wheel_back">
+    <link name="right_wheel_rear">
         <visual>
             <geometry>
@@ -133,3 +147,8 @@
         </xacro:inertial_cylinder>
     </link>
+    <gazebo reference="right_wheel_rear">
+        <material>Gazebo/Blue</material>
+        <mu1 value="0.001"/>
+        <mu2 value="0.001"/>
+    </gazebo>
 </robot>

Commit message: new commit

File: description/robot.urdf.xacro (robot description, xacro)
@@ -3,3 +3,4 @@
     <xacro:include filename="robot_core.xacro" />
     <xacro:include filename="gazebo_control.xacro" />
+    <xacro:include filename="lidar.xacro" />
 </robot>

File: description/robot_core.xacro (robot description, xacro)
@@ -13,4 +13,7 @@
     <material name ="black">
         <color rgba="0 0 0 1" />
+    </material>
+    <material name ="red">
+        <color rgba="1 0 0 1" />
     </material>
     <!-- BASE LINK -->
